File: ESP_S3_MONITOR/V_1_2/Pcb FIle/ESP S3 _ MONITOR_V_1_2.kicad_pcb (KiCad board)
At the start: 2 copper layers, 82 x 50 mm, 79 parts, among them J1 USB_C_Receptacle_USB2.0_16P, J2 Screw_Terminal_01x03, J3 Battery Connector, J4 Conn_01x04_Socket, J5 Conn_01x09_Socket, J6 Conn_02x03_Top_Bottom, J7 Conn_02x06_Top_Bottom, K1 Songle SRD-03VDC-SL-C, Q1 BC817, Q2 AO3401A, Q3 BC817, Q4 AO3401A, Q6 AO3400A, U1 AHT20, U2 PC817, U3 USBLC6-2SC6, U4 ESP32-S3-WROOM-1, U5 BQ24040DSQR, U6 TPS631000DRLR, U7 RA-01H, U8 SCD40-D-R2

Commit message: Some update
Parts:
- added BT2: BK-912, BK-912:BAT_BK-912, F.Cu at (38.0, 50.8)
- added C11: 18pF, Capacitor_SMD:C_0805_2012Metric_Pad1.18x1.45mm_HandSolder, F.Cu at (51.2, 62.0)
- added C12: 18pF, Capacitor_SMD:C_0805_2012Metric_Pad1.18x1.45mm_HandSolder, F.Cu at (51.2, 65.0)
- added C13: 100nF, Capacitor_SMD:C_0805_2012Metric_Pad1.18x1.45mm_HandSolder, F.Cu at (51.2, 68.0)
- added D8: SS14, Diode_SMD:D_SMA, F.Cu at (28.9, 62.8)
- added D9: SS14, Diode_SMD:D_SMA, F.Cu at (28.9, 67.3)
- added R38: 4.7K, Resistor_SMD:R_0805_2012Metric_Pad1.20x1.40mm_HandSolder, F.Cu at (53.5, 42.6)
- added R39: 4.7K, Resistor_SMD:R_0805_2012Metric_Pad1.20x1.40mm_HandSolder, F.Cu at (53.5, 45.6)
- added R40: 4.7K, Resistor_SMD:R_0805_2012Metric_Pad1.20x1.40mm_HandSolder, F.Cu at (53.5, 48.5)
- added U11: ABS25-32.768KHZ-1-T, ul_ABS25-32-768KHZ-1-T:ABS25-32.768KHZ-1-T_ABR, F.Cu at (36.9, 65.3)
- added U12: PCF8563T_F4_118, PCF8563T_F4_118:SOIC127P600X175-8N, F.Cu at (44.8, 63.5)
