File: ESP_S3_MONITOR/V_1_2/Pcb FIle/_autosave-ESP S3 _ MONITOR.kicad_pcb (KiCad board)
At the start: 2 copper layers, 82 x 50 mm, 79 parts, among them J1 USB_C_Receptacle_USB2.0_16P, J2 Screw_Terminal_01x03, J3 Battery Connector, J4 Conn_01x04_Socket, J5 Conn_01x09_Socket, J6 Conn_02x03_Top_Bottom, J7 Conn_02x06_Top_Bottom, K1 Songle SRD-03VDC-SL-C, Q1 BC817, Q2 AO3401A, Q3 BC817, Q4 AO3401A, Q6 AO3400A, U1 AHT20, U2 PC817, U3 USBLC6-2SC6, U4 ESP32-S3-WROOM-1, U5 BQ24040DSQR, U6 TPS631000DRLR, U7 RA-01H, U8 SCD40-D-R2

Commit message: Some update
Parts:
- added BT1: BK-912, BK-912:BAT_BK-912, F.Cu at (35.6, 55.7)
- added D6: SS14, Diode_SMD:D_SMA, F.Cu at (34.4, 67.7)
- added D7: SS14, Diode_SMD:D_SMA, F.Cu at (34.4, 72.2)
- added R35: 4.7K, Resistor_SMD:R_0805_2012Metric_Pad1.20x1.40mm_HandSolder, F.Cu at (40.8, 66.9)
- added R36: 4.7K, Resistor_SMD:R_0805_2012Metric_Pad1.20x1.40mm_HandSolder, F.Cu at (40.8, 69.8)
- added R37: 4.7K, Resistor_SMD:R_0805_2012Metric_Pad1.20x1.40mm_HandSolder, F.Cu at (40.8, 72.8)
- added U10: ABS25-32.768KHZ-1-T, ul_ABS25-32-768KHZ-1-T:ABS25-32.768KHZ-1-T_ABR, F.Cu at (26.4, 70.2)
- added U9: PCF8563T_F4_118, PCF8563T_F4_118:SOIC127P600X175-8N, F.Cu at (47.2, 68.4)
