File: ESP_S3_MONITOR/V_1_0/Pcb FIle/ESP S3 _ MONITOR.kicad_pcb (KiCad board)
At the start: 2 copper layers, 82 x 50 mm, 79 parts, among them J1 USB_C_Receptacle_USB2.0_16P, J2 Screw_Terminal_01x03, J3 Battery Connector, J4 Conn_01x04_Socket, J5 Conn_01x09_Socket, J6 Conn_02x03_Top_Bottom, J7 Conn_02x06_Top_Bottom, K1 Songle SRD-03VDC-SL-C, Q1 BC817, Q2 AO3401A, Q3 BC817, Q4 AO3401A, Q6 AO3400A, U1 AHT20, U2 PC817, U3 USBLC6-2SC6, U4 ESP32-S3-WROOM-1, U5 BQ24040DSQR, U6 TPS631000DRLR, U7 RA-01H, U8 SCD40-D-R2

Commit message: Some update
Changed lines of the file:
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@@
 			(unlocked yes)
 			(layer "F.SilkS")
+			(hide yes)
 			(effects
 				(font
@@
 			(unlocked yes)
 			(layer "F.Fab")
+			(hide yes)
 			(effects
 				(font
@@
 			(layer "F.Fab")
 		)
-		(fp_text user "${REFERENCE}"
-			(at 0 0 180)
-			(unlocked yes)
-			(layer "F.Fab")
-			(effects
-				(font
-					(size 1 1)
-					(thickness 0.15)
-				)
-			)
-		)
 		(pad "1" smd rect
 			(at -0.8001 -0.750001 180)
@@
 		)
 		(embedded_fonts no)
+		(model "${KIPRJMOD}/EG1247/EG1247.step"
+			(offset
+				(xyz 0 0 1)
+			)
+			(scale
+				(xyz 1 1 1)
+			)
+			(rotate
+				(xyz -90 -0 90)
+			)
+		)
 	)
 	(footprint "Package_TO_SOT_SMD:SOT-23"
@@
 		)
 		(embedded_fonts no)
-		(model "${KICAD9_3DMODEL_DIR}/Connector_USB.3dshapes/USB_C_Receptacle_G-Switch_GT-USB-7010ASV.step"
+		(model "D:/pcb-portfolio/USB SO_SIN/V_1_0/Step File/CQ-USB-C16PSMT01.step"
 			(offset
 				(xyz 0 0 0)
@@
 			)
 			(rotate
-				(xyz 0 0 0)
+				(xyz -90 -0 -0)
 			)
 		)
