File: FT234XD/V_1_0/Pcb File/FT234XD.kicad_pcb (KiCad board)
At the start: 2 copper layers, 11 parts, among them J2 USB_A, Q2 AO3401A, U1 FT234XD, U3 USBLC6-2SC6

Commit message: Some update
Parts:
- added C4: 1 uF, Capacitor_SMD:C_0805_2012Metric_Pad1.18x1.45mm_HandSolder, F.Cu at (68.4, 45.3)
- added C5: 10uF, Capacitor_SMD:C_0805_2012Metric_Pad1.18x1.45mm_HandSolder, B.Cu at (82.7, 56.9)
- added D1: LED, LED_SMD:LED_0805_2012Metric_Pad1.15x1.40mm_HandSolder, F.Cu at (61.2, 15.3)
- added D2: LED, LED_SMD:LED_0805_2012Metric_Pad1.15x1.40mm_HandSolder, F.Cu at (58.1, 58.5)
- added D4: LED, LED_SMD:LED_0805_2012Metric_Pad1.15x1.40mm_HandSolder, F.Cu at (61.2, 21.4)
- added J1: Conn_01x06, Connector_PinSocket_2.54mm:PinSocket_1x06_P2.54mm_Vertical, F.Cu at (86.8, 43.9)
- added J3: Conn_02x03_Counter_Clockwise, Connector_PinSocket_2.54mm:PinSocket_2x03_P2.54mm_Vertical_SMD, F.Cu at (78.7, 46.5)
- added Q1: SS8050, Package_TO_SOT_SMD:SOT-23, F.Cu at (79.7, 57.2)
- added Q3: SS8050, Package_TO_SOT_SMD:SOT-23, F.Cu at (79.7, 53.2)
- added R1: 220R, Resistor_SMD:R_0805_2012Metric_Pad1.20x1.40mm_HandSolder, F.Cu at (76.3, 55.2)
- added R15: 330R, Resistor_SMD:R_0805_2012Metric_Pad1.20x1.40mm_HandSolder, F.Cu at (54.7, 17.6)
- added R16: 330R, Resistor_SMD:R_0805_2012Metric_Pad1.20x1.40mm_HandSolder, F.Cu at (65.9, 21.2)
- added R2: 220R, Resistor_SMD:R_0805_2012Metric_Pad1.20x1.40mm_HandSolder, F.Cu at (73.9, 55.2)
- added R5: 330R, Resistor_SMD:R_0805_2012Metric_Pad1.20x1.40mm_HandSolder, F.Cu at (62.2, 58.5)
- added R6: 10K, Resistor_SMD:R_0805_2012Metric_Pad1.20x1.40mm_HandSolder, F.Cu at (1.88, 3.98)
- added U2: CP2102N-Axx-xQFN20, Package_DFN_QFN:SiliconLabs_QFN-20-1EP_3x3mm_P0.5mm_EP1.8x1.8mm, F.Cu at (68.1, 50.2)
- C3: value 100 nF -> 10uF
- U1: value FT234XD -> AP2112K-3.3; footprint Package_DFN_QFN:WDFN-12-1EP_3x3mm_P0.45mm_EP1.7x2.5mm -> Package_TO_SOT_SMD:SOT-23-5
- moved C2 74.4 mm to (58.2, 45.3), turned to 90 degrees
- moved U1 71.1 mm to (62.0, 45.4), turned to 0 degrees
- moved FB1 70.4 mm to (57.1, 55.1), turned to -90 degrees
- moved C3 69.5 mm to (65.7, 45.3), turned to -90 degrees
- moved J2 63.5 mm to (43.5, 50.5)
- moved R4 63.4 mm to (58.2, 51.5)
- moved R3 63.4 mm to (58.2, 49.5)
- moved U3 63.3 mm to (62.9, 50.4)
- moved R14 61.8 mm to (66.0, 55.1), turned to -90 degrees
- moved C1 61.2 mm to (59.5, 55.1), turned to 90 degrees
- moved Q2 61.1 mm to (62.8, 55.1), turned to -90 degrees
Connections:
- C1 pad 1: Net-(J2-VBUS) -> Net-(Q2-D)
- C3 pad 1: /3.3V -> 3.3V
- FB1 pad 1: Net-(Q2-S) -> Net-(J2-VBUS)
- FB1 pad 2: VBUS -> Net-(Q2-D)
- Q2 pad 2: Net-(Q2-S) -> VBUS
- Q2 pad 3: Net-(J2-VBUS) -> Net-(Q2-D)
- U1 pad 1: /D- -> VBUS
- U1 pad 3: /3.3V -> VBUS
- U1 pad 4: VBUS -> unconnected-(U1-NC-Pad4)
- U1 pad 5: GND -> 3.3V
- U3 pad 5: Net-(J2-VBUS) -> Net-(Q2-D)
Routing:
- net Net-(Q2-D): track 0.00 -> 10.9 mm, vias 0 -> 3
- net VBUS: track 2.16 -> 12.5 mm, vias 0 -> 2
- net Net-(J2-VBUS): track 12.6 -> 3.05 mm
- net ESP_IO0: track 0.00 -> 6.50 mm
- net ESP_EN: track 0.00 -> 6.40 mm
- net /D+: track 0.00 -> 3.77 mm
- net Net-(Q2-G): track 5.95 -> 2.29 mm
- net Net-(Q2-S): track 3.29 -> 0.00 mm
- net /D-: track 0.00 -> 2.74 mm
- net GND: track 0.00 -> 2.33 mm, vias 0 -> 2
- net Net-(D2-A): track 0.00 -> 2.03 mm
- added copper zone on B.Cu, net GND
- added copper zone on F.Cu, net GND
Other:
- board outline added: 40 x 20 mm
- board text added: "3.3V"
