File: SM_CON_PCB/V_1_0/Pcb File/SM_C_PCB.kicad_sch (KiCad schematic)
At the start: 9 parts, among them J3 USB_C_Receptacle_USB2.0_16P, U1 ATtiny10-TS

Commit message: Some update
Parts:
- R2: value 330K -> 330R
Connections:
- net RESET: now reaches R1.1, U1.6 (~{RESET}/PB3)
Changed lines of the file:
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@@
+		)
+	)
+	(bus
+		(pts
+			(xy 16.51 85.09) (xy 16.51 17.78)
+		)
+		(stroke
+			(width 0)
+			(type dash_dot_dot)
 		)
 	)
@@
 		)
 	)
+	(bus
+		(pts
+			(xy 16.51 17.78) (xy 181.61 17.78)
+		)
+		(stroke
+			(width 0)
+			(type dash_dot_dot)
+		)
+	)
+	(bus
+		(pts
+			(xy 181.61 17.78) (xy 181.61 85.09)
+		)
+		(stroke
+			(width 0)
+			(type dash_dot_dot)
+		)
+	)
 	(wire
 		(pts
@@
 			(width 0)
 			(type default)
+		)
+	)
+	(bus
+		(pts
+			(xy 181.61 85.09) (xy 16.51 85.09)
+		)
+		(stroke
+			(width 0)
+			(type dash_dot_dot)
 		)
 	)
@@
 	(label "CC2"
 		(at 57.15 36.83 0)
+		(effects
+			(font
+				(size 1.27 1.27)
+			)
+			(justify left bottom)
+		)
+	)
+	(label "RESET"
+		(at 130.81 48.26 0)
 		(effects
 			(font
@@
 			)
 		)
-		(property "Value" "330K"
+		(property "Value" "330R"
 			(at 153.67 41.91 90)
 			(effects
